File: sesame.kicad_pcb (KiCad board)
At the start: 2 copper layers, 344.4 x 130.9 mm, 165 parts, among them U1 ATmega32A-PU

Commit message: add stepped caps support
Parts:
- added MX69: MX-NoLED, MX_Only:MXOnly-1.25U-NoLED, F.Cu at (79.1, 127.5)
- MX59: footprint MX_Only:MXOnly-1.75U-NoLED -> MX_Only:MXOnly-1.5U-NoLED
Connections:
- net Net-(D34-Pad2) renamed caps
Routing:
- net caps: track 12.2 -> 26.9 mm
- net col1: track 211.0 -> 219.6 mm

Commit message: minor design changes
Parts:
- removed the REF** at (211.9, 92.3)
- removed the REF** at (139.3, 76.3)
- removed the REF** at (282.1, 76.3)
- added AVR1: Conn_01x06, Connector_PinHeader_2.54mm:PinHeader_1x06_P2.54mm_Vertical, F.Cu at (227.7, 66.9)
- added REF**: screw_hole, custom_parts:screw_hole, F.Cu at (279.0, 75.6)
- added REF**: screw_hole, custom_parts:screw_hole, F.Cu at (142.4, 75.6)
- C1: footprint Capacitor_THT:CP_Radial_D5.0mm_P2.50mm -> Capacitor_THT:CP_Radial_D4.0mm_P1.50mm
- MX15: footprint MX_Only:MXOnly-2.25U-NoLED -> MX_Only:MXOnly-2U-NoLED
- MX31: footprint MX_Only:MXOnly-1U-NoLED -> MX_Only:MXOnly-1.5U-NoLED
- MX59: footprint MX_Only:MXOnly-1.5U-NoLED -> MX_Only:MXOnly-1.75U-NoLED
- MX61: footprint MX_Only:MXOnly-2.25U-NoLED -> MX_Only:MXOnly-2.75U-NoLED
- moved D17 26.1 mm to (372.2, 93.4), turned to 90 degrees
- moved F1 2.25 mm to (147.8, 78.0), turned to 348 degrees
- moved C1 0.55 mm to (150.3, 74.0), turned to 12 degrees
Routing:
- net row0: track 320.0 -> 342.2 mm
- net VCC: track 28.5 -> 16.5 mm
- net bs: track 26.1 -> 19.5 mm
- net SCK: track 0.00 -> 6.04 mm
- net MOSI: track 0.00 -> 6.04 mm
- net MISO: track 0.00 -> 6.04 mm
- net reset: track 65.2 -> 71.2 mm
- net +5V: track 146.2 -> 145.7 mm
Other:
- board text added: "GND"
- board text added: "MISO"
- board text added: "MOSI"
- board text added: "RST"
- board text added: "SCK"
- board text added: "VCC"

Commit message: fix routing error
Connections:
- net boot renamed BOOT
- net reset renamed RST
Routing:
- net col13: track 223.7 -> 225.0 mm

Commit message: update gerbers to latest kicad version defaults
Other:
- rule pad_to_mask_clearance: 0.05 -> 0
