File: sesame.kicad_pcb (KiCad board)
At the start: 2 copper layers, 344.4 x 130.9 mm, 166 parts, among them U1 ATmega32A-PU

Commit message: add 2.25u left space support and update caps to use cftkb footprints
Parts:
- added MX70: MX-NoLED, MX_Only:MXOnly-2.25U-ReversedStabilizers-NoLED, F.Cu at (166.6, 174.0)
- added MX71: MX-NoLED, MX_Only:MXOnly-1U-NoLED, F.Cu at (196.9, 180.5)
- MX62, MX63: footprint MX_Only:MXOnly-1U-NoLED -> MX_Only:MXOnly-1.5U-NoLED
- moved D64 1.48 mm to (183.6, 181.7)
- moved C3 1.36 mm to (206.3, 88.2)
- moved C2 1.28 mm to (211.5, 66.9)
- moved C4 1.12 mm to (240.6, 84.8)
- moved C5 1.12 mm to (240.6, 69.0)
- renumbered R3 to R2, R2 to R3
Routing:
- net col6: track 109.8 -> 112.2 mm
- net col5: track 123.4 -> 125.7 mm
- net Net-(D64-Pad2): track 16.6 -> 18.3 mm
- net +5V: track 145.7 -> 144.3 mm
- net GND: track 11.5 -> 12.4 mm
- net Net-(C5-Pad2): track 43.5 -> 42.9 mm
- net Net-(C4-Pad2): track 49.1 -> 48.5 mm
- added copper zone on B.Cu, net Net-(D64-Pad2)
- added copper zone on B.Cu, net Net-(D65-Pad2)
- added copper zone on F.Cu, net col5
- added copper zone on F.Cu, net col6

Commit message: fixes
Parts:
- C2, C3: footprint Capacitor_THT:C_Disc_D3.0mm_W2.0mm_P2.50mm -> Capacitor_THT:C_Disc_D5.0mm_W2.5mm_P5.00mm
- C4, C5: footprint Capacitor_THT:C_Disc_D6.0mm_W2.5mm_P5.00mm -> Capacitor_THT:C_Disc_D5.0mm_W2.5mm_P2.50mm
Other:
- board text added: "Sesame Ergo PCB rev. 2 github.com/kb-elmo/sesame elmo.space"
- board text removed: "Sesame Ergo PCB rev. 1 github.com/kb-elmo/sesame elmo.space"
